File: KiCad_v2/SignaLink.kicad_pcb (KiCad board)
At the start: 2 copper layers, 60 x 45 mm, 68 parts, among them Q1 MMBT3904, SW1 SW_Wake, U1 DM-OLED096-636, U2 ESP32-C3_SUPERMINI_TH, U3 MIC94063YC6-TR, U4 CM4102008, U5 LT8582EDKD-PBF, U6 MCP73871, U7 LM3940IMP-3.3, U8 BNO085, U9 MPU-6050

Commit message: modificaciones en silkscreen
Parts:
- D2: renamed from D1; value LED-MCP -> LED
- D3: renamed from D2; value LED-MCP -> LED
- D4: renamed from D3; value LED-MCP -> LED
- R5: renamed from R5-MIC1; value 100k -> 4k7
- moved SW1 1.88 mm to (25.9, 85.8)
- moved G*** 0.09 mm to (41.9, 53.6)
- renumbered C18-LT1 to C10, C19-LT1 to C11, C2 to C12, C3 to C13, C4-BNO1 to C14, C9-BNO1 to C15, C3-BNO1 to C16, C4-MPU1 to C17, C5-MPU1 to C18, C6-MPU1 to C19, C16-LT1 to C2, C7-MPU1 to C20, C13-LT1 to C3, C15-LT1 to C4, C7-MCP1 to C5, C17-LT1 to C6, C8-MCP1 to C7, C14-LT1 to C8, C10-MCP1 to C9, D4-LT1 to D1, L1-LT1 to L1, L2-LT1 to L2, R8-LT1 to R10, R12-MCP1 to R11, R11-MCP1 to R12, R1-LT1 to R13, R20-LT1 to R14, R10-MCP1 to R15, R6-MCP1 to R16, R7-MCP1 to R17, R9-LT1 to R18, R15-BNO1 to R19, R19-BNO1 to R20, R18-BNO1 to R21, R14-BNO1 to R22, R9-MPU1 to R23, R10-MPU1 to R24, R3-MIC1 to R3, R13-MCP1 to R9
Routing:
- net GND: track 408.1 -> 409.8 mm
- net Net-(U4A-GPIO2): track 61.0 -> 62.2 mm

Commit message: feat: sumo usb c y edito esquematico
Parts:
- added J1: USB_C_Receptacle, Connector_USB:USB_C_Receptacle_G-Switch_GT-USB-7010ASV, F.Cu at (33.4, 88.2)
- added R25: R, Resistor_SMD:R_0603_1608Metric, F.Cu at (22.0, 81.8)
- added R26: R, Resistor_SMD:R_0603_1608Metric, F.Cu at (37.8, 82.4)
- moved SW1 7.45 mm to (20.9, 91.3), turned to 90 degrees
- moved S1 1.63 mm to (74.6, 83.0)
- moved S2 1.62 mm to (74.6, 76.6)
- moved S4 1.60 mm to (74.6, 63.6)
- moved S3 1.60 mm to (74.6, 70.1)
- moved G*** 0.20 mm to (63.8, 81.7)
- moved G*** 0.20 mm to (41.9, 53.8)
Connections:
- U4 pad 103: unconnected-(U4B-USB_N-Pad103) -> /USB_N
- U4 pad 105: unconnected-(U4B-USB_P-Pad105) -> /USB_P
Routing:
- net /USB_N: track 0.00 -> 20.1 mm, vias 0 -> 1
- net Net-(J1-CC1): track 0.00 -> 16.9 mm, vias 0 -> 2
- net /USB_P: track 0.00 -> 14.2 mm, vias 0 -> 3
- net GND: track 409.8 -> 422.8 mm
- net Net-(U4A-GPIO2): track 62.2 -> 73.9 mm
- net +3.3V: track 163.7 -> 171.2 mm
- net +5V: track 189.7 -> 195.6 mm
- net Net-(J1-CC2): track 0.00 -> 3.64 mm
- net /A4: track 31.2 -> 33.9 mm
- net /A2: track 27.5 -> 29.1 mm
- net /A3: track 29.6 -> 31.1 mm

Commit message: feat: Cambios FINALES de la placa
Subo version final
Parts:
- R25, R26: value R -> 5k1
- moved U2 2.06 mm to (58.3, 61.0)
Connections:
- U2 pad 5: /A5 -> unconnected-(U2-GPIO5-Pad5)
Routing:
- net /A2: track 29.1 -> 33.5 mm
- net /A1: track 30.7 -> 35.1 mm
- net +3.3V: track 171.2 -> 167.7 mm
- net /A4: track 33.9 -> 36.8 mm
- net /A3: track 31.1 -> 34.0 mm
- net GND: track 422.8 -> 425.6 mm
- net /SCL: track 92.6 -> 94.3 mm
- net /SDA: track 85.0 -> 86.4 mm
- net /USB_N: track 20.1 -> 21.5 mm
- net /MIC_OUT: track 17.4 -> 16.1 mm
- net /USB_PORT: track 64.0 -> 63.0 mm
- net Net-(U5-RT1): track 23.3 -> 24.1 mm
- net +5V: track 195.6 -> 195.1 mm
- net Net-(MOLEX1-Pin_1): track 16.0 -> 16.5 mm
- added copper zone on B.Cu, net GND
- added copper zone on F.Cu, net GND

Commit message: feat: FINAL
Parts:
- removed SW1: SW_Wake, Button_Switch_THT:SW_Tactile_Straight_KSA0Axx1LFTR
- added S5: ~, Custom_Footprints:PULSADOR, F.Cu at (22.8, 87.4)
- C10, C11: footprint Capacitor_SMD:C_0603_1608Metric -> Custom_Footprints:CAP_6TPB68M
- L1, L2: footprint Custom_Footprints:IND_SRP6540-100M -> Custom_Footprints:COILSR
- S1, S2, S3, S4: footprint Connector_Molex:Molex_KK-254_AE-6410-02A_1x02_P2.54mm_Vertical -> Connector_Molex:Molex_Signalink
- moved C11 12.8 mm to (19.6, 74.0), turned to 90 degrees
- moved C10 8.65 mm to (22.0, 78.7), turned to 180 degrees
- moved D1 3.01 mm to (28.5, 79.3)
- moved L2 0.33 mm to (23.6, 73.6)
Routing:
- net GND: track 425.6 -> 454.7 mm
- net +3.3V: track 167.7 -> 192.3 mm
- net Net-(U4A-GPIO2): track 73.4 -> 65.5 mm
- net /A1: track 35.1 -> 27.9 mm
- net Net-(J1-CC1): track 16.9 -> 21.9 mm, vias 2 -> 0
- net /A4: track 36.8 -> 33.9 mm
- net +5V: track 195.1 -> 197.5 mm
- net Net-(C6-Pad2): track 21.2 -> 22.6 mm, vias 0 -> 2
- net Net-(U5-SWA1): track 18.4 -> 19.4 mm
- net /A2: track 33.5 -> 32.6 mm
- net Net-(C10-Pad2): track 2.97 -> 3.59 mm
- net /power_supply/OUT_MCP: track 67.2 -> 67.7 mm
Other:
- board size 60 x 45 mm -> 61.5 x 45 mm

Commit message: este si es el final
Parts:
- moved S4 1.26 mm to (74.5, 62.3)
- moved S2 1.26 mm to (74.5, 75.3)
- moved S1 1.26 mm to (74.5, 81.7)
- moved S3 1.26 mm to (74.5, 68.8)
- moved C1 0.65 mm to (63.6, 52.6)
- moved R8 0.65 mm to (65.4, 52.6)
Routing:
- net +3.3V: track 192.3 -> 184.3 mm
- net /A3: track 33.7 -> 32.5 mm
- net /A4: track 33.9 -> 33.1 mm
- net Net-(U4A-GLOBAL_EN): track 6.96 -> 7.66 mm
- net GND: track 454.7 -> 455.3 mm
- net /A1: track 27.9 -> 27.4 mm
