File: KiCad_v2/giroscopos.kicad_sch (KiCad schematic)
At the start: 15 parts, among them U8 BNO085, U9 MPU-6050

Commit message: modificaciones en silkscreen
Parts:
- renumbered C4-BNO1 to C14, C9-BNO1 to C15, C3-BNO1 to C16, C4-MPU1 to C17, C5-MPU1 to C18, C6-MPU1 to C19, C7-MPU1 to C20, R15-BNO1 to R19, R19-BNO1 to R20, R18-BNO1 to R21, R14-BNO1 to R22, R9-MPU1 to R23, R10-MPU1 to R24
Other:
- moved on the sheet: R20

Commit message: feat: Cambios FINALES de la placa
Subo version final
Changed lines of the file:
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@@
-	(wire
-		(pts
-			(xy 214.63 148.59) (xy 228.6 148.59)
-		)
-		(stroke
-			(width 0)
-			(type default)
-		)
-	)
 	(wire
 		(pts
@@
 	(label "SDA"
 		(at 201.93 83.82 0)
-		(effects
-			(font
-				(size 1.27 1.27)
-			)
-			(justify left bottom)
-		)
-	)
-	(label "A5"
-		(at 214.63 148.59 0)
 		(effects
 			(font
@@
 		(effects
 			(font
-				(size 1.27 1.27)
-			)
-			(justify left)
-		)
-	)
-	(hierarchical_label "A5"
-		(shape input)
-		(at 228.6 148.59 0)
-		(effects
-			(font
