File: KiCad_v2/SignaLink.kicad_sch (KiCad schematic)
At the start: 19 parts, among them Q1 MMBT3904, SW1 SW_Wake, U1 DM-OLED096-636, U2 ESP32-C3_SUPERMINI_TH, U3 MIC94063YC6-TR, U4 CM4102008

Commit message: feat: arreglos en pistas y correcciones de errores
Other:
- moved on the sheet: R3-MIC1
Changed lines of the file:
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@@
 	(wire
 		(pts
-			(xy 45.72 123.19) (xy 46.99 123.19)
-		)
-		(stroke
-			(width 0)
-			(type default)
-		)
-	)
-	(wire
-		(pts
 			(xy 115.57 30.48) (xy 119.38 30.48)
 		)
@@
 	(wire
 		(pts
-			(xy 45.72 110.49) (xy 46.99 110.49)
-		)
-		(stroke
-			(width 0)
-			(type default)
-		)
-	)
-	(wire
-		(pts
 			(xy 48.26 26.67) (xy 46.99 26.67)
 		)
@@
 	(wire
 		(pts
-			(xy 46.99 110.49) (xy 46.99 107.95)
-		)
-		(stroke
-			(width 0)
-			(type default)
-		)
-	)
-	(wire
-		(pts
 			(xy 60.96 26.67) (xy 60.96 30.48)
 		)
@@
 	(wire
 		(pts
-			(xy 46.99 123.19) (xy 46.99 127)
+			(xy 45.72 118.11) (xy 49.53 118.11)
 		)
 		(stroke
@@
 	(wire
 		(pts
-			(xy 45.72 118.11) (xy 49.53 118.11)
+			(xy 73.66 152.4) (xy 63.5 152.4)
 		)
 		(stroke
@@
 	(wire
 		(pts
-			(xy 73.66 152.4) (xy 63.5 152.4)
+			(xy 55.88 60.96) (xy 66.04 60.96)
 		)
 		(stroke
@@
 	(wire
 		(pts
-			(xy 109.22 182.88) (xy 109.22 173.99)
-		)
-		(stroke
-			(width 0)
-			(type default)
-		)
-	)
-	(wire
-		(pts
 			(xy 46.99 24.13) (xy 48.26 24.13)
 		)
@@
 	(wire
 		(pts
-			(xy 40.64 171.45) (xy 46.99 171.45)
+			(xy 44.45 171.45) (xy 46.99 171.45)
 		)
 		(stroke
@@
 	(wire
 		(pts
-			(xy 59.69 86.36) (xy 55.88 86.36)
+			(xy 109.22 176.53) (xy 109.22 173.99)
 		)
 		(stroke
@@
 	(wire
 		(pts
-			(xy 60.96 38.1) (xy 60.96 40.64)
+			(xy 59.69 86.36) (xy 55.88 86.36)
 		)
 		(stroke
@@
 	(wire
 		(pts
-			(xy 55.88 60.96) (xy 60.96 60.96)
+			(xy 60.96 38.1) (xy 60.96 40.64)
 		)
 		(stroke
@@
 		)
 	)
+	(wire
+		(pts
+			(xy 109.22 176.53) (xy 118.11 176.53)
+		)
+		(stroke
+			(width 0)
+			(type default)
+		)
+	)
 	(label "GND"
 		(at -57.15 60.96 0)
@@
 	)
 	(label "MIC_OUT"
-		(at 109.22 182.88 90)
+		(at 118.11 176.53 180)
 		(effects
 			(font
 				(size 1.27 1.27)
 			)
-			(justify left bottom)
+			(justify right bottom)
 		)
 	)
@@
 	)
 	(label "MIC_OUT"
-		(at 60.96 60.96 0)
+		(at 66.04 60.96 180)
 		(effects
 			(font
 				(size 1.27 1.27)
 			)
-			(justify left bottom)
+			(justify right bottom)
 		)
 	)
@@
 	(symbol
 		(lib_id "power:+3.3V")
-		(at 33.02 171.45 90)
+		(at 36.83 171.45 90)
 		(unit 1)
 		(exclude_from_sim no)
@@
 		(fields_autoplaced yes)
 		(property "Reference" "#PWR03"
-			(at 36.83 171.45 0)
+			(at 40.64 171.45 0)
 			(effects
 				(font
@@
 		)
 		(property "Value" "+3.3V"
-			(at 29.21 171.4499 90)
+			(at 33.02 171.4499 90)
 			(effects
 				(font
@@
 		)
 		(property "Footprint" ""
-			(at 33.02 171.45 0)
+			(at 36.83 171.45 0)
 			(effects
 				(font
@@
 		)
 		(property "Datasheet" ""
-			(at 33.02 171.45 0)
+			(at 36.83 171.45 0)
 			(effects
 				(font
@@
 		)
 		(property "Description" "Power symbol creates a global label with name \"+3.3V\""
-			(at 33.02 171.45 0)
+			(at 36.83 171.45 0)
 			(effects
 				(font
@@
 	(symbol
 		(lib_id "power:+3V3")
-		(at 46.99 107.95 0)
+		(at 45.72 110.49 270)
 		(unit 1)
 		(exclude_from_sim no)
@@
 		(fields_autoplaced yes)
 		(property "Reference" "#PWR06"
-			(at 46.99 111.76 0)
+			(at 41.91 110.49 0)
 			(effects
 				(font
@@
 		)
 		(property "Value" "+3.3V"
-			(at 46.99 102.87 0)
+			(at 49.53 110.4899 90)
 			(effects
 				(font
 					(size 1.27 1.27)
 				)
+				(justify left)
 			)
 		)
 		(property "Footprint" ""
-			(at 46.99 107.95 0)
+			(at 45.72 110.49 0)
 			(effects
 				(font
@@
 		)
 		(property "Datasheet" ""
-			(at 46.99 107.95 0)
+			(at 45.72 110.49 0)
 			(effects
 				(font
@@
 		)
 		(property "Description" "Power symbol creates a global label with name \"+3V3\""
-			(at 46.99 107.95 0)
+			(at 45.72 110.49 0)
 			(effects
 				(font
@@
 	(symbol
 		(lib_id "power:GND")
-		(at 46.99 127 0)
+		(at 45.72 123.19 90)
 		(unit 1)
 		(exclude_from_sim no)
@@
 		(fields_autoplaced yes)
 		(property "Reference" "#PWR07"
-			(at 46.99 133.35 0)
+			(at 52.07 123.19 0)
 			(effects
 				(font
@@
 		)
 		(property "Value" "GND"
-			(at 46.99 132.08 0)
+			(at 49.53 123.1899 90)
 			(effects
 				(font
 					(size 1.27 1.27)
 				)
+				(justify right)
 			)
 		)
 		(property "Footprint" ""
-			(at 46.99 127 0)
+			(at 45.72 123.19 0)
 			(effects
 				(font
@@
 		)
 		(property "Datasheet" ""
-			(at 46.99 127 0)
+			(at 45.72 123.19 0)
 			(effects
 				(font
@@
 		)
 		(property "Description" "Power symbol creates a global label with name \"GND\" , ground"
-			(at 46.99 127 0)
+			(at 45.72 123.19 0)
 			(effects
 				(font
@@
 	(symbol
 		(lib_id "Device:R")
-		(at 36.83 171.45 90)
+		(at 40.64 171.45 90)
 		(unit 1)
 		(exclude_from_sim no)
@@
 		(fields_autoplaced yes)
 		(property "Reference" "R3-MIC1"
-			(at 36.83 165.1 90)
+			(at 40.64 165.1 90)
 			(effects
 				(font
@@
 		)
 		(property "Value" "100k"
-			(at 36.83 167.64 90)
+			(at 40.64 167.64 90)
 			(effects
 				(font
@@
 		)
 		(property "Footprint" "Resistor_SMD:R_0603_1608Metric"
-			(at 36.83 173.228 90)
+			(at 40.64 173.228 90)
 			(effects
 				(font
@@
 		)
 		(property "Datasheet" "~"
-			(at 36.83 171.45 0)
+			(at 40.64 171.45 0)
 			(effects
 				(font
@@
 		)
 		(property "Description" "Resistor"
-			(at 36.83 171.45 0)
+			(at 40.64 171.45 0)
 			(effects
 				(font
@@
 		)
 		(property "Field4" ""
-			(at 36.83 171.45 90)
+			(at 40.64 171.45 90)
 			(effects
 				(font
@@
 		)
 		(property "Field5" ""
-			(at 36.83 171.45 90)
+			(at 40.64 171.45 90)
 			(effects
 				(font

Commit message: feat: subo version final del pcb y sumo logos
Parts:
- R5-MIC1: value 100k -> 4k7
Other:
- sheet power_supply ports: added none; removed 5V
Changed lines of the file:
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@@
 	(wire
 		(pts
-			(xy -57.15 57.15) (xy -49.53 57.15)
-		)
-		(stroke
-			(width 0)
-			(type default)
-		)
-	)
-	(wire
-		(pts
 			(xy 22.86 26.67) (xy 26.67 26.67)
 		)
@@
 		)
 	)
-	(label "5V"
-		(at -57.15 57.15 0)
-		(effects
-			(font
-				(size 1.27 1.27)
-			)
-			(justify left bottom)
-		)
-	)
 	(label "A4"
 		(at 64.77 26.67 180)
@@
 			)
 		)
-		(property "Value" "100k"
+		(property "Value" "4k7"
 			(at 59.69 148.59 90)
 			(effects
@@
 			)
 		)
-		(pin "5V" input
-			(at -49.53 57.15 180)
-			(effects
-				(font
-					(size 1.27 1.27)
-				)
-				(justify left)
-			)
-		)

Commit message: modificaciones en silkscreen
Parts:
- renumbered R3-MIC1 to R3, R5-MIC1 to R5
Changed lines of the file:
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@@
 		(dnp no)
 		(fields_autoplaced yes)
-		(property "Reference" "#PWR05"
+		(property "Reference" "#PWR04"
 			(at 35.56 46.99 0)
 			(effects
@@
 			(project "SignaLink"
 				(path "/a1f5fcc2-f8ff-418d-9afd-dd6d7b5c6dc3"
-					(reference "#PWR05")
+					(reference "#PWR04")
 					(unit 1)
 				)
@@
 		(dnp no)
 		(fields_autoplaced yes)
-		(property "Reference" "R5-MIC1"
+		(property "Reference" "R5"
 			(at 59.69 146.05 90)
 			(effects
@@
 			(project ""
 				(path "/a1f5fcc2-f8ff-418d-9afd-dd6d7b5c6dc3"
-					(reference "R5-MIC1")
+					(reference "R5")
 					(unit 1)
 				)
@@
 		(dnp no)
 		(fields_autoplaced yes)
-		(property "Reference" "#PWR03"
+		(property "Reference" "#PWR05"
 			(at 40.64 171.45 0)
 			(effects
@@
 			(project ""
 				(path "/a1f5fcc2-f8ff-418d-9afd-dd6d7b5c6dc3"
-					(reference "#PWR03")
+					(reference "#PWR05")
 					(unit 1)
 				)
@@
 		(dnp no)
 		(fields_autoplaced yes)
-		(property "Reference" "#PWR04"
+		(property "Reference" "#PWR03"
 			(at 35.56 25.4 0)
 			(effects
@@
 			(project "SignaLink"
 				(path "/a1f5fcc2-f8ff-418d-9afd-dd6d7b5c6dc3"
-					(reference "#PWR04")
+					(reference "#PWR03")
 					(unit 1)
 				)
@@
 		(dnp no)
 		(fields_autoplaced yes)
-		(property "Reference" "R3-MIC1"
+		(property "Reference" "R3"
 			(at 40.64 165.1 90)
 			(effects
@@
 			(project ""
 				(path "/a1f5fcc2-f8ff-418d-9afd-dd6d7b5c6dc3"
-					(reference "R3-MIC1")
+					(reference "R3")
 					(unit 1)
 				)

Commit message: feat: sumo usb c y edito esquematico
Parts:
- added J1: USB_C_Receptacle, Connector_USB:USB_C_Receptacle_G-Switch_GT-USB-7010ASV, symbol Connector:USB_C_Receptacle
- added R25, R26: 5k1, Resistor_SMD:R_0603_1608Metric, symbol Device:R
Connections:
- net +5V: now also J1.A4 (VBUS), J1.A9 (VBUS), J1.B4 (VBUS), J1.B9 (VBUS)
- net GND: now also J1.A1 (GND), J1.A12 (GND), J1.B1 (GND), J1.B12 (GND), J1.S1 (SHIELD), R25.2, R26.2
- net USB_N: now reaches U4.103 (USB_N)
- net USB_N: now also J1.B6 (D+), J1.B7 (D-)
- net USB_P: now reaches U4.105 (USB_P)
- net USB_P: now also J1.A6 (D+), J1.A7 (D-)
- new net: J1.A5 (CC1), R25.1
- new net: J1.B5 (CC2), R26.1

Commit message: feat: Cambios FINALES de la placa
Subo version final
Connections:
- net A5: no longer names the net of U2.5 (GPIO5)
- no-connect marks 143 -> 144
Other:
- sheet giroscopos ports: added none; removed A5
Changed lines of the file:
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@@
 	)
 	(no_connect
+		(at 20.32 78.74)
+	)
+	(no_connect
 		(at 280.67 53.34)
 	)
@@
 	(wire
 		(pts
-			(xy -58.42 66.04) (xy -49.53 66.04)
-		)
-		(stroke
-			(width 0)
-			(type default)
-		)
-	)
-	(wire
-		(pts
 			(xy 48.26 24.13) (xy 48.26 21.59)
 		)
@@
 	(wire
 		(pts
-			(xy -60.96 96.52) (xy -49.53 96.52)
-		)
-		(stroke
-			(width 0)
-			(type default)
-		)
-	)
-	(wire
-		(pts
 			(xy 48.26 30.48) (xy 48.26 26.67)
 		)
@@
 	(wire
 		(pts
-			(xy 109.22 176.53) (xy 109.22 173.99)
+			(xy -59.69 63.5) (xy -49.53 63.5)
 		)
 		(stroke
@@
 	(wire
 		(pts
-			(xy 59.69 86.36) (xy 55.88 86.36)
+			(xy 109.22 176.53) (xy 109.22 173.99)
 		)
 		(stroke
@@
 	(wire
 		(pts
-			(xy 60.96 38.1) (xy 60.96 40.64)
+			(xy 59.69 86.36) (xy 55.88 86.36)
 		)
 		(stroke
@@
 	(wire
 		(pts
-			(xy 35.56 26.67) (xy 39.37 26.67)
+			(xy 60.96 38.1) (xy 60.96 40.64)
 		)
 		(stroke
@@
 	(wire
 		(pts
-			(xy 15.24 78.74) (xy 20.32 78.74)
+			(xy 35.56 26.67) (xy 39.37 26.67)
 		)
 		(stroke
@@
 		)
 	)
-	(label "A5"
-		(at 15.24 78.74 0)
-		(effects
-			(font
-				(size 1.27 1.27)
-			)
-			(justify left bottom)
-		)
-	)
-	(label "A5"
-		(at -60.96 96.52 0)
-		(effects
-			(font
-				(size 1.27 1.27)
-			)
-			(justify left bottom)
-		)
-	)
 	(label "GND"
 		(at 115.57 30.48 0)
@@
 	)
 	(label "USB_PORT"
-		(at -58.42 66.04 0)
+		(at -59.69 63.5 0)
 		(effects
 			(font
@@
 			)
 		)
-		(pin "A5" input
-			(at -49.53 96.52 180)
-			(effects
-				(font
-					(size 1.27 1.27)
-				)
-				(justify left)
-			)
-		)
 		(pin "SCL" input
 			(at -49.53 93.98 180)
@@
 		)
 		(pin "USB" input
-			(at -49.53 66.04 180)
+			(at -49.53 63.5 180)
 			(effects
 				(font

Commit message: feat: FINAL
Parts:
- removed SW1: SW_Wake, Button_Switch_THT:SW_Tactile_Straight_KSA0Axx1LFTR, symbol Switch:SW_Push
- added S5: ~, Custom_Footprints:PULSADOR, symbol PULSADOR:TS11-674-43-BK-100-RA-D
- S1, S2, S3, S4: footprint Connector_Molex:Molex_KK-254_AE-6410-02A_1x02_P2.54mm_Vertical -> Connector_Molex:Molex_Signalink
Connections:
- net GND: now also S5.2, S5.3 (GND), S5.4 (GND)
- net at R7.2, U4.58 (GPIO2): now also S5.1
Other:
- moved on the sheet: R7
