File: KiCad_v2/power_supply.kicad_sch (KiCad schematic)
At the start: 32 parts, among them U5 LT8582EDKD-PBF, U6 MCP73871, U7 LM3940IMP-3.3

Commit message: feat: subo version final del pcb y sumo logos
Connections:
- net 5V is gone; now on net +5V: U6.17 (CE), U6.3 (SEL), U6.4 (PROG2), U6.9 (~{TE})

Commit message: modificaciones en silkscreen
Parts:
- D2: renamed from D1; value LED-MCP -> LED
- D3: renamed from D2; value LED-MCP -> LED
- D4: renamed from D3; value LED-MCP -> LED
- renumbered C18-LT1 to C10, C19-LT1 to C11, C2 to C12, C3 to C13, C16-LT1 to C2, C13-LT1 to C3, C15-LT1 to C4, C7-MCP1 to C5, C17-LT1 to C6, C8-MCP1 to C7, C14-LT1 to C8, C10-MCP1 to C9, D4-LT1 to D1, L1-LT1 to L1, L2-LT1 to L2, R8-LT1 to R10, R12-MCP1 to R11, R11-MCP1 to R12, R1-LT1 to R13, R20-LT1 to R14, R10-MCP1 to R15, R6-MCP1 to R16, R7-MCP1 to R17, R9-LT1 to R18, R13-MCP1 to R9

Commit message: feat: FINAL
Parts:
- C10, C11: footprint Capacitor_SMD:C_0603_1608Metric -> Custom_Footprints:CAP_6TPB68M
- L1, L2: footprint Custom_Footprints:IND_SRP6540-100M -> Custom_Footprints:COILSR
Changed lines of the file:
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@@
 			)
 		)
-		(property "Footprint" "Custom_Footprints:IND_SRP6540-100M"
+		(property "Footprint" "Custom_Footprints:COILSR"
 			(at 57.15 109.22 0)
 			(effects
@@
 			)
 		)
-		(property "Footprint" "Capacitor_SMD:C_0603_1608Metric"
+		(property "Footprint" "Custom_Footprints:CAP_6TPB68M"
 			(at 147.0152 132.08 0)
 			(effects
@@
 			)
 		)
-		(property "Footprint" "Capacitor_SMD:C_0603_1608Metric"
+		(property "Footprint" "Custom_Footprints:CAP_6TPB68M"
 			(at 147.0152 121.92 0)
 			(effects
@@
 			)
 		)
-		(property "Footprint" "Custom_Footprints:IND_SRP6540-100M"
+		(property "Footprint" "Custom_Footprints:COILSR"
 			(at 86.36 113.03 0)
 			(effects
